File: PCB/kicad/sensors.kicad_sch (KiCad schematic)
At the start: 30 parts

Commit message: Added some test points
Parts:
- added TP2: TestPoint, TestPoint:TestPoint_Pad_D1.0mm, symbol Connector:TestPoint
Connections:
- net AN_IIN: now also TP2.1
Changed lines of the file:
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@@
   (junction (at 83.82 140.97) (diameter 0) (color 0 0 0 0)
+  )
+  (junction (at 92.71 143.51) (diameter 0) (color 0 0 0 0)
   )
   (junction (at 72.39 86.36) (diameter 0) (color 0 0 0 0)
@@
     (stroke (width 0) (type default))
   )
-  (wire (pts (xy 77.47 143.51) (xy 91.44 143.51))
+  (wire (pts (xy 77.47 143.51) (xy 92.71 143.51))
     (stroke (width 0) (type default))
   )
@@
     (stroke (width 0) (type default))
   )
+  (wire (pts (xy 171.45 154.94) (xy 190.5 154.94))
+    (stroke (width 0) (type default))
+  )
+  (wire (pts (xy 92.71 143.51) (xy 95.25 143.51))
+    (stroke (width 0) (type default))
+  )
   (wire (pts (xy 214.63 67.31) (xy 214.63 69.85))
     (stroke (width 0) (type default))
@@
   )
   (wire (pts (xy 68.58 86.36) (xy 72.39 86.36))
-    (stroke (width 0) (type default))
-  )
-  (wire (pts (xy 171.45 154.94) (xy 190.5 154.94))
     (stroke (width 0) (type default))
   )
@@
     )
   )
-  (global_label "AN_IIN" (shape output) (at 91.44 143.51 0) (fields_autoplaced)
+  (global_label "AN_IIN" (shape output) (at 95.25 143.51 0) (fields_autoplaced)
     (effects (font (size 1 1)) (justify left))
-    (property "Intersheetrefs" "${INTERSHEET_REFS}" (at 98.3945 143.51 0)
+    (property "Intersheetrefs" "${INTERSHEET_REFS}" (at 102.2045 143.51 0)
       (effects (font (size 1.27 1.27)) (justify left) hide)
     )
@@
         )
       )
+    )
+  )
+  (symbol (lib_id "Connector:TestPoint") (at 92.71 143.51 0) (unit 1)
+    (in_bom yes) (on_board yes) (dnp no)
+    (property "Reference" "TP2" (at 95.25 137.16 0)
+      (effects (font (size 1.27 1.27)) (justify right))
+    )
+    (property "Value" "TestPoint" (at 90.17 138.938 0)
+      (effects (font (size 1.27 1.27)) (justify right) hide)
+    )
+    (property "Footprint" "TestPoint:TestPoint_Pad_D1.0mm" (at 97.79 143.51 0)
+      (effects (font (size 1.27 1.27)) hide)
+    )
+    (property "Datasheet" "~" (at 97.79 143.51 0)
+      (effects (font (size 1.27 1.27)) hide)
+    )
+    (pin "1")
+    (instances
+      (project "smartplug"
+        (path "/85f97cef-95fb-4a05-880a-b699f4dd7284/eaa7450d-3a78-4f54-b267-5efe8ce0cdad"
+          (reference "TP2") (unit 1)
+        )
+        (path "/85f97cef-95fb-4a05-880a-b699f4dd7284/5e43e972-422a-4dae-8dd2-68614bca60dd"
+          (reference "TP2") (unit 1)
+        )
+      )
